File: prominifinal.brd (EAGLE design)
At the start: 74.6 x 50.8 mm, 9 parts, among them IC1 EL357N-B-TA-G

Commit message: GND edit
Connections:
- removed net N$24: 1.9, D2.C, PROMINI.GND
- net N$26: now also 1.9, D2.C, PROMINI.GND
Routing:
- net N$26: track 141.6 -> 257.6 mm, vias 1 -> 2
- net N$24: track 98.6 -> 0.00 mm, vias 1 -> 0
Changed lines of the file:
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@@
 <wire x1="3.81" y1="32.385" x2="3.47" y2="32.83" width="0.762" layer="16"/>
-</signal>
-<signal name="N$24">
-<contactref element="PROMINI" pad="GND"/>
-<contactref element="1" pad="9"/>
-<contactref element="D2" pad="C"/>
-<wire x1="28.575" y1="17.145" x2="28.575" y2="46.99" width="0.762" layer="1"/>
-<wire x1="39.37" y1="7.62" x2="38.1" y2="7.62" width="0.762" layer="1"/>
-<wire x1="38.1" y1="7.62" x2="28.575" y2="17.145" width="0.762" layer="1"/>
-<wire x1="41.275" y1="7.62" x2="39.37" y2="7.62" width="0.762" layer="16"/>
-<wire x1="44.45" y1="4.445" x2="41.275" y2="7.62" width="0.762" layer="16"/>
-<wire x1="44.45" y1="3.81" x2="44.45" y2="4.445" width="0.762" layer="16"/>
-<wire x1="28.575" y1="46.99" x2="28.98" y2="46.99" width="0.762" layer="1"/>
-<via x="39.37" y="7.62" extent="1-16" drill="0.5"/>
-<wire x1="60.96" y1="16.51" x2="61.957" y2="15.513" width="0.762" layer="1"/>
-<wire x1="61.957" y1="15.513" x2="61.957" y2="15.2168625" width="0.762" layer="1"/>
-<wire x1="69.85" y1="7.3238625" x2="69.85" y2="1.397" width="0.762" layer="1"/>
-<wire x1="61.957" y1="15.2168625" x2="69.85" y2="7.3238625" width="0.762" layer="1"/>
-<wire x1="69.85" y1="1.397" x2="44.45" y2="1.397" width="0.762" layer="1"/>
-<wire x1="44.45" y1="1.397" x2="44.45" y2="3.81" width="0.762" layer="1"/>
 </signal>
 <signal name="N$26">
@@
 <wire x1="3.175" y1="30.48" x2="3.47" y2="30.33" width="0.762" layer="16"/>
 <via x="30.48" y="33.655" extent="1-16" drill="0.5"/>
+<contactref element="PROMINI" pad="GND"/>
+<contactref element="1" pad="9"/>
+<contactref element="D2" pad="C"/>
+<wire x1="28.575" y1="17.145" x2="28.575" y2="46.99" width="0.762" layer="1"/>
+<wire x1="39.37" y1="7.62" x2="38.1" y2="7.62" width="0.762" layer="1"/>
+<wire x1="38.1" y1="7.62" x2="28.575" y2="17.145" width="0.762" layer="1"/>
+<wire x1="41.275" y1="7.62" x2="39.37" y2="7.62" width="0.762" layer="16"/>
+<wire x1="44.45" y1="4.445" x2="41.275" y2="7.62" width="0.762" layer="16"/>
+<wire x1="44.45" y1="3.81" x2="44.45" y2="4.445" width="0.762" layer="16"/>
+<wire x1="28.575" y1="46.99" x2="28.98" y2="46.99" width="0.762" layer="1"/>
+<via x="39.37" y="7.62" extent="1-16" drill="0.5"/>
+<wire x1="60.96" y1="16.51" x2="61.957" y2="15.513" width="0.762" layer="1"/>
+<wire x1="61.957" y1="15.513" x2="61.957" y2="15.2168625" width="0.762" layer="1"/>
+<wire x1="69.85" y1="7.3238625" x2="69.85" y2="1.397" width="0.762" layer="1"/>
+<wire x1="61.957" y1="15.2168625" x2="69.85" y2="7.3238625" width="0.762" layer="1"/>
+<wire x1="69.85" y1="1.397" x2="44.45" y2="1.397" width="0.762" layer="1"/>
+<wire x1="44.45" y1="1.397" x2="44.45" y2="3.81" width="0.762" layer="1"/>
+<wire x1="60.96" y1="26.035" x2="60.96" y2="16.51" width="0.762" layer="1"/>
+<wire x1="55.88" y1="31.115" x2="60.96" y2="26.035" width="0.762" layer="1"/>
+<wire x1="55.88" y1="31.75" x2="55.88" y2="31.115" width="0.762" layer="1"/>
 </signal>
 <signal name="N$4">
