File: prominifinal.sch (EAGLE design)
At the start: 9 parts, among them IC1 EL357N-B-TA-G

Commit message: GND edit
Connections:
- removed net N$24: 1.9, D2.C, PROMINI.GND
- net N$26: now also 1.9, D2.C, PROMINI.GND
Changed lines of the file:
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@@
-</segment>
-</net>
-<net name="N$24" class="0">
-<segment>
-<pinref part="PROMINI" gate="G$1" pin="GND"/>
-<wire x1="116.84" y1="72.39" x2="137.16" y2="72.39" width="0.762" layer="91"/>
-<wire x1="137.16" y1="72.39" x2="137.16" y2="71.12" width="0.762" layer="91"/>
-<pinref part="1" gate="A" pin="9"/>
-<wire x1="137.16" y1="71.12" x2="137.16" y2="-11.43" width="0.762" layer="91"/>
-<wire x1="137.16" y1="-11.43" x2="165.1" y2="-11.43" width="0.762" layer="91"/>
-<pinref part="D2" gate="G$1" pin="C"/>
-<wire x1="166.37" y1="53.34" x2="166.37" y2="71.12" width="0.762" layer="91"/>
-<wire x1="166.37" y1="71.12" x2="137.16" y2="71.12" width="0.762" layer="91"/>
-<junction x="137.16" y="71.12"/>
 </segment>
 </net>
@@
 <wire x1="86.14" y1="125.08" x2="86.14" y2="125.73" width="0.762" layer="91"/>
 <wire x1="86.14" y1="125.73" x2="71.12" y2="125.73" width="0.762" layer="91"/>
-<wire x1="71.12" y1="125.73" x2="71.12" y2="100.33" width="0.762" layer="91"/>
+<wire x1="71.12" y1="125.73" x2="71.12" y2="116.84" width="0.762" layer="91"/>
+<wire x1="71.12" y1="116.84" x2="71.12" y2="100.33" width="0.762" layer="91"/>
 <wire x1="71.12" y1="100.33" x2="60.96" y2="100.33" width="0.762" layer="91"/>
 <pinref part="D1" gate="G$1" pin="C"/>
@@
 <wire x1="2.54" y1="118.11" x2="2.54" y2="110.49" width="0.762" layer="91"/>
 <junction x="60.96" y="100.33"/>
+<pinref part="PROMINI" gate="G$1" pin="GND"/>
+<wire x1="116.84" y1="72.39" x2="137.16" y2="72.39" width="0.762" layer="91"/>
+<wire x1="137.16" y1="72.39" x2="137.16" y2="71.12" width="0.762" layer="91"/>
+<pinref part="1" gate="A" pin="9"/>
+<wire x1="137.16" y1="71.12" x2="137.16" y2="-11.43" width="0.762" layer="91"/>
+<wire x1="137.16" y1="-11.43" x2="165.1" y2="-11.43" width="0.762" layer="91"/>
+<pinref part="D2" gate="G$1" pin="C"/>
+<wire x1="166.37" y1="53.34" x2="166.37" y2="71.12" width="0.762" layer="91"/>
+<wire x1="166.37" y1="71.12" x2="160.02" y2="71.12" width="0.762" layer="91"/>
+<junction x="137.16" y="71.12"/>
+<wire x1="160.02" y1="71.12" x2="137.16" y2="71.12" width="0.762" layer="91"/>
+<wire x1="71.12" y1="116.84" x2="160.02" y2="116.84" width="0.762" layer="91"/>
+<wire x1="160.02" y1="116.84" x2="160.02" y2="71.12" width="0.762" layer="91"/>
+<junction x="71.12" y="116.84"/>
+<junction x="160.02" y="71.12"/>
 </segment>
 </net>

Commit message: final
Parts:
- removed D1: RED, SparkFun-LED:LED-RED1206
Connections:
- new net N$15: 2.10, PROMINI.D8
- net N$1: no longer 2.10, D1.A
- net N$26: no longer D1.C
Changed lines of the file:
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@@
 <part name="1" library="pinhead" deviceset="PINHD-1X10" device=""/>
 <part name="DIODE" library="adafruit" deviceset="DIODE" device="SOD-323F"/>
-<part name="D1" library="SparkFun-LED" deviceset="LED-RED" device="1206" value="RED"/>
 <part name="U$1" library="SIM800LMODULE" deviceset="SIM800LMODULE" device=""/>
 <part name="VCC-GND" library="SparkFun-Retired" deviceset="CONN_02" device="5MM"/>
@@
 <attribute name="VALUE" x="53.34" y="132.08" size="1.27" layer="96"/>
 </instance>
-<instance part="D1" gate="G$1" x="48.26" y="105.41" smashed="yes">
-<attribute name="NAME" x="44.831" y="100.838" size="1.778" layer="95" font="vector" rot="R90"/>
-<attribute name="VALUE" x="50.165" y="100.838" size="1.778" layer="96" font="vector" rot="R90" align="top-left"/>
-</instance>
 <instance part="U$1" gate="G$1" x="104.14" y="132.08" smashed="yes"/>
 <instance part="VCC-GND" gate="G$1" x="-10.16" y="118.11" smashed="yes">
@@
 <net name="N$1" class="0">
 <segment>
-<wire x1="2.54" y1="125.73" x2="12.7" y2="125.73" width="0.762" layer="91"/>
-<wire x1="12.7" y1="125.73" x2="22.86" y2="125.73" width="0.762" layer="91"/>
+<wire x1="2.54" y1="125.73" x2="22.86" y2="125.73" width="0.762" layer="91"/>
 <wire x1="22.86" y1="125.73" x2="22.86" y2="113.03" width="0.762" layer="91"/>
 <wire x1="43.18" y1="113.03" x2="43.18" y2="135.89" width="0.762" layer="91"/>
 <wire x1="43.18" y1="135.89" x2="53.34" y2="135.89" width="0.762" layer="91"/>
-<wire x1="43.18" y1="113.03" x2="48.26" y2="113.03" width="0.762" layer="91"/>
-<wire x1="48.26" y1="113.03" x2="48.26" y2="107.95" width="0.762" layer="91"/>
-<junction x="48.26" y="113.03"/>
-<wire x1="48.26" y1="113.03" x2="111.76" y2="113.03" width="0.762" layer="91"/>
+<wire x1="43.18" y1="113.03" x2="129.54" y2="113.03" width="0.762" layer="91"/>
 <pinref part="DIODE" gate="G$1" pin="A"/>
-<pinref part="D1" gate="G$1" pin="A"/>
 <wire x1="22.86" y1="113.03" x2="43.18" y2="113.03" width="0.762" layer="91"/>
 <junction x="43.18" y="113.03"/>
-<pinref part="2" gate="A" pin="10"/>
-<wire x1="50.8" y1="24.13" x2="50.8" y2="-16.51" width="0.762" layer="91"/>
-<wire x1="50.8" y1="-16.51" x2="15.24" y2="-16.51" width="0.762" layer="91"/>
-<wire x1="12.7" y1="125.73" x2="12.7" y2="24.13" width="0.762" layer="91"/>
-<wire x1="12.7" y1="24.13" x2="50.8" y2="24.13" width="0.762" layer="91"/>
-<junction x="12.7" y="125.73"/>
 <pinref part="VCC-GND" gate="G$1" pin="2"/>
 <wire x1="-2.54" y1="120.65" x2="2.54" y2="120.65" width="0.762" layer="91"/>
 <wire x1="2.54" y1="120.65" x2="2.54" y2="125.73" width="0.762" layer="91"/>
-<wire x1="111.76" y1="113.03" x2="129.54" y2="113.03" width="0.762" layer="91"/>
 <wire x1="129.54" y1="113.03" x2="129.54" y2="74.93" width="0.762" layer="91"/>
 <pinref part="PROMINI" gate="G$1" pin="RAW"/>
@@
 <wire x1="71.12" y1="116.84" x2="71.12" y2="100.33" width="0.762" layer="91"/>
 <wire x1="71.12" y1="100.33" x2="60.96" y2="100.33" width="0.762" layer="91"/>
-<pinref part="D1" gate="G$1" pin="C"/>
-<junction x="48.26" y="100.33"/>
-<wire x1="60.96" y1="100.33" x2="48.26" y2="100.33" width="0.762" layer="91"/>
-<wire x1="48.26" y1="100.33" x2="22.86" y2="100.33" width="0.762" layer="91"/>
+<wire x1="60.96" y1="100.33" x2="22.86" y2="100.33" width="0.762" layer="91"/>
 <wire x1="22.86" y1="110.49" x2="22.86" y2="100.33" width="0.762" layer="91"/>
 <wire x1="2.54" y1="110.49" x2="22.86" y2="110.49" width="0.762" layer="91"/>
@@
 </segment>
 </net>
+<net name="N$15" class="0">
+<segment>
+<pinref part="PROMINI" gate="G$1" pin="D8"/>
+<wire x1="76.2" y1="49.53" x2="53.34" y2="49.53" width="0.762" layer="91"/>
+<wire x1="53.34" y1="49.53" x2="53.34" y2="-17.78" width="0.762" layer="91"/>
+<wire x1="53.34" y1="-17.78" x2="15.24" y2="-17.78" width="0.762" layer="91"/>
+<pinref part="2" gate="A" pin="10"/>
+<wire x1="15.24" y1="-17.78" x2="15.24" y2="-16.51" width="0.762" layer="91"/>
+</segment>
+</net>
